Commit message: Add robot

File: limo_car/gazebo/ackermann_with_sensor.xacro (robot description, xacro)
@@ -8,4 +8,5 @@
 <robot name="limo_ackermann" xmlns:xacro="http://www.ros.org/wiki/xacro">
     <xacro:include filename="$(find limo_car)/gazebo/ackermann.xacro" />
+    <xacro:limo_ackermann />
     <xacro:include filename="$(find limo_car)/gazebo/sensor.xacro" />
     <!-- ************************* Laser ****************************** -->

File: limo_car/gazebo/four_diff.xacro (robot description, xacro)
@@ -8,5 +8,5 @@
 dargestellt. Es erhält sich noch die Funktionen über Reglung für Lenkung und Bewegung, wie die in Gazebo realisiert werden.
 Es würde einfach in andere Datei angerufen werden. -->
-<robot name="limo_ackermann" xmlns:xacro="http://www.ros.org/wiki/xacro">
+<robot name="limo_four_diff" xmlns:xacro="http://www.ros.org/wiki/xacro">
     <!-- ******************************** Paramenten zu definieren ************************************* -->
     <!-- *********************************************************************************************** -->
@@ -73,5 +73,6 @@
             </collision>
         </link>
-        <joint name="${wheel_prefix}_steer_joint" type="revolute">
+        <!-- Four-diff mode: keep the front wheel pointing straight. -->
+        <joint name="${wheel_prefix}_steer_joint" type="fixed">
             <parent link="${parent_prefix}"/>
             <child link="${wheel_prefix}_steer_link"/>
@@ -146,5 +147,6 @@
             </collision>
         </link>
-        <joint name="${wheel_prefix}_steer_joint" type="revolute">
+        <!-- Four-diff mode: keep the front wheel pointing straight. -->
+        <joint name="${wheel_prefix}_steer_joint" type="fixed">
             <parent link="${parent_prefix}"/>
             <child link="${wheel_prefix}_steer_link"/>
@@ -203,5 +205,5 @@
     <!-- erstellt Hauptanteil des Modells, definiert ein Nullpunkt, um Modell aufzubauen. Es ist einfach für weitere
     Darstellungspostion in Simulation-Umgebung -->
-    <xacro:macro name="limo_ackermann">
+    <xacro:macro name="limo_four_diff">
         <!-- <link name="base_footprint"/>
         <joint name="base_joint" type="fixed">
@@ -306,18 +308,27 @@
         <!-- *********************************************************************************************** -->
         <gazebo>
-            <!--
-              The upstream Ackermann setup does not drive this small LIMO model
-              reliably on Gazebo 11 / ROS 2 Humble. Use the ROS 2 planar plugin
-              for stable map, sensor and navigation testing.
-            -->
-            <plugin name="limo_planar_controller" filename="libgazebo_ros_planar_move.so">
+            <!-- Four-wheel skid-steer drive: both wheels on each side receive
+                 the same velocity command from gazebo_ros_diff_drive. -->
+            <plugin name="limo_four_diff_controller" filename="libgazebo_ros_diff_drive.so">
                 <ros>
                     <remapping>cmd_vel:=/cmd_vel</remapping>
                     <remapping>odom:=/odom</remapping>
                 </ros>
-                <update_rate>100.0</update_rate>
+                <update_rate>100</update_rate>
+                <num_wheel_pairs>2</num_wheel_pairs>
+                <left_joint>front_left_wheel_joint</left_joint>
+                <left_joint>rear_left_wheel_joint</left_joint>
+                <right_joint>front_right_wheel_joint</right_joint>
+                <right_joint>rear_right_wheel_joint</right_joint>
+                <wheel_separation>${track}</wheel_separation>
+                <wheel_separation>${track}</wheel_separation>
+                <wheel_diameter>${2 * wheel_radius}</wheel_diameter>
+                <wheel_diameter>${2 * wheel_radius}</wheel_diameter>
+                <max_wheel_torque>20.0</max_wheel_torque>
+                <max_wheel_acceleration>5.0</max_wheel_acceleration>
                 <publish_rate>50.0</publish_rate>
                 <publish_odom>true</publish_odom>
                 <publish_odom_tf>true</publish_odom_tf>
+                <publish_wheel_tf>true</publish_wheel_tf>
                 <odometry_frame>odom</odometry_frame>
                 <robot_base_frame>base_link</robot_base_frame>

File: limo_car/gazebo/sensor.xacro (robot description, xacro)
@@ -143,5 +143,5 @@
                     </ros>
                     <camera_name>${frame_prefix}</camera_name>
-                    <frame_name>${frame_prefix}_frame_optical</frame_name>
+                    <frame_name>${frame_prefix}_link</frame_name>
                     <hack_baseline>0.07</hack_baseline>
                     <min_depth>0.001</min_depth>
